File: hw/christmas_ornament.kicad_sch (KiCad schematic)
At the start: 23 parts, among them J1 AVR-UPDI-6, U1 ATtiny404-SS, U3 ST25DV04K-IER6T3

Commit message: update
Connections:
- net I2C_SCL: now also U3.6 (SCL); no longer U3.2 (AC0)
- net I2C_SDA: now also U3.5 (SDA); no longer U3.1 (V_EH)
- net NFC_INT: now also U3.7 (GPO); no longer U3.3 (AC1)
- net V_EH: now also U3.1 (V_EH); no longer U3.5 (SDA)
- net at AE1.1, C2.1, C3.2: now also U3.2 (AC0); no longer U3.6 (SCL)
- net at AE1.2, C2.2, C4.1: now also U3.3 (AC1); no longer U3.7 (GPO)
Changed lines of the file:
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@@
 		(lib_id "christmas_ornament_sym_lib:ST25DV04K-IER6T3")
 		(at 153.67 139.7 0)
+		(mirror y)
 		(unit 1)
 		(exclude_from_sim no)
@@
 		(fields_autoplaced yes)
 		(property "Reference" "U3"
-			(at 155.8641 129.54 0)
+			(at 151.4759 129.54 0)
 			(effects
 				(font
@@
 		)
 		(property "Value" "ST25DV04K-IER6T3"
-			(at 155.8641 132.08 0)
+			(at 151.4759 132.08 0)
 			(effects
 				(font
